File: Amiga600.sch (KiCad schematic (older format))
At the start: 40 parts, among them U1 MC68000, U2 AGNUS, U21 74LS245, U22 74LS245, U5 GAYLE

Commit message: Add files via upload
A slightly modified design, that removes the RF modulator and fits an S-Video connector in the space. It utilises the CXA2075 video encoder to create the S-video output and removes the need for the bandpass and delay lines.

This design has been tested and is working.
Parts:
- removed ER199: *, Resistor_SMD:R_1206_3216Metric_Pad1.42x1.75mm_HandSolder, symbol Device:Ferrite_Bead_Small
- removed XC1: 0.33uF, Capacitor_SMD:C_1206_3216Metric_Pad1.42x1.75mm_HandSolder, symbol Device:C_Small
- removed XJA1, XJB1, XJC1: Jumper, Jumper:SolderJumper-2_P1.3mm_Bridged_Pad1.0x1.5mm, symbol Device:Jumper_NC_Small
- removed XU1: PAL16L8B, Package_DIP:DIP-20_W7.62mm, symbol MyLibrary:PAL16L8B
- added E199: 27, MyLibrary:SMD_1206, symbol Device:R_Small
- added ER131: 68, MyLibrary:SMD_1206, symbol Device:R_Small
- added U25: 74F258, MyLibrary:SOIC-16-DUAL, symbol MyLibrary:74F258
- added X1: 28.37516MHz, MyLibrary:Oscillator, symbol MyLibrary:28.37516MHz
- EC112: value 22 -> 22pF; footprint Capacitor_SMD:C_1206_3216Metric_Pad1.42x1.75mm_HandSolder -> MyLibrary:SMD_1206; symbol Device:R_Small -> Device:C_Small
- EC120: value 0.22UF -> 0.33uF; footprint Capacitor_SMD:C_1206_3216Metric_Pad1.42x1.75mm_HandSolder -> MyLibrary:SMD_1206
- EC121: value 22 -> *; footprint Capacitor_SMD:C_1206_3216Metric_Pad1.42x1.75mm_HandSolder -> MyLibrary:SMD_1206
- EC122, EC123, EC124, EC125, EC126, EC127: value 22 -> 22pF; footprint Capacitor_SMD:C_1206_3216Metric_Pad1.42x1.75mm_HandSolder -> MyLibrary:SMD_1206
- EC128, EC129: value 22 -> 47pF; footprint Capacitor_SMD:C_1206_3216Metric_Pad1.42x1.75mm_HandSolder -> MyLibrary:SMD_1206
- ER112, ER120, ER121, ER122, ER123, ER124, ER125, ER128, ER129, ER132, R101, R102, R103, R111, R113, R114: footprint Resistor_SMD:R_1206_3216Metric_Pad1.42x1.75mm_HandSolder -> MyLibrary:SMD_1206
- ER126, ER127: value 27 -> 47; footprint Resistor_SMD:R_1206_3216Metric_Pad1.42x1.75mm_HandSolder -> MyLibrary:SMD_1206
- U1: footprint Package_LCC:PLCC-68 -> MyLibrary:PLCC-68
- U2, U5: footprint Package_LCC:PLCC-84 -> MyLibrary:PLCC-84
- U21, U22: footprint Package_SO:SOIC-20W_7.5x12.8mm_P1.27mm -> MyLibrary:SOIC-20W
Connections:
- net labels added: +5V, XCLK, _XCLKEN
- net labels removed: U1_14, U1_16, U1_17, U1_18, U1_31, U1_52, U1_56, U1_57, U21_10, U21_20, U22_10, U22_20, U25_12, U2_15, U2_41, U2_58, U2_82, U5_1, U5_12, U5_13, U5_14, U5_18, U5_19, U5_2, U5_20, U5_24, U5_3, U5_4, U5_45, U5_5, U5_6, U5_62, U5_63, U5_64, U5_65, U5_66, U5_67, U5_68, U5_69, U5_7, U5_70, U5_71, U5_72, U5_75, U5_76, U5_77, U5_78, U5_79, U5_8, U5_80, U5_81, U5_83, U5_84, U5_9, VCC, XU1_10, XU1_20, _IDE_CS[1], _IDE_CS[2]
- wire segments 379 -> 339
- no-connect marks 2 -> 9
Other:
- note added: "Note: NTSC uses 28.63636MHz"
- note added: "Note: Various components are for EMI Control\nand may be loaded with funny things..."
- moved on the sheet: EC120, EC121, EC122, EC123, EC124, EC125, EC126, EC127, EC128, EC129, ER112, ER120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
