File: Sheet10.sch (KiCad schematic (older format))
At the start: 34 parts, among them CN15 PCMCIA, U41 74LS245, U42 74LS245, U43 74LS245, U44 74F02, U45 74LS245, U46 74LS245, U47 74LS245

Commit message: Add files via upload
A slightly modified design, that removes the RF modulator and fits an S-Video connector in the space. It utilises the CXA2075 video encoder to create the S-video output and removes the need for the bandpass and delay lines.

This design has been tested and is working.
Parts:
- removed XJD1, XJE1: Jumper, Jumper:SolderJumper-2_P1.3mm_Bridged_Pad1.0x1.5mm, symbol Device:Jumper_NC_Small
- added unit 2 of U41
- added unit 2 of U42
- added unit 2 of U43
- added unit 4 of U44
- added unit 5 of U44
- added unit 2 of U44
- added unit 1 of U44
- added unit 2 of U45
- added unit 2 of U46
- added unit 2 of U47
- added U5: GAYLE, MyLibrary:PLCC-84, symbol MyLibrary:GAYLE
- C41, C42, C43, C44, C45, C46, C47, C701, C702, C711: footprint Capacitor_SMD:C_1210_3225Metric_Pad1.42x2.65mm_HandSolder -> MyLibrary:SMD_1210
- R716, R717, R718, RA714, RA715, RB714, RB715, RC715, RD715, RE715, RF715, RG715, RX715, RY715: footprint Resistor_SMD:R_1206_3216Metric_Pad1.42x1.75mm_HandSolder -> MyLibrary:SMD_1206
- U41, U42, U43, U45, U46, U47: footprint Package_SO:SOIC-20W_7.5x12.8mm_P1.27mm -> MyLibrary:SOIC-20W
- U44: footprint Package_SO:SOIC-14_3.9x8.7mm_P1.27mm -> MyLibrary:SOIC-14
Connections:
- net labels added: +5V, VPP
- net labels removed: U41_10, U41_20, U42_10, U42_20, U43_10, U43_20, U44_14, U44_7, U45_10, U45_20, U46_10, U46_20, U47_10, U47_20, U5_1, U5_12, U5_13, U5_14, U5_18, U5_19, U5_2, U5_4, U5_5, U5_6, U5_7, U5_75, U5_76, U5_77, U5_78, U5_79, U5_8, U5_80, U5_81, U5_83, U5_84, U5_9, VCC, Vpp
- wire segments 446 -> 395
- no-connect marks 3 -> 5
Other:
- note added: "SPARE"
- note added: "Warning:\nByte Swapped"
- moved on the sheet: C41, C42, C43, C44, C45, C46, C47, C702, C711, R718, RA714, RA715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
