File: Sheet11.sch (KiCad schematic (older format))
At the start: 3 parts, among them CN16 IDE, P9 80PIN

Commit message: Add files via upload
A slightly modified design, that removes the RF modulator and fits an S-Video connector in the space. It utilises the CXA2075 video encoder to create the S-video output and removes the need for the bandpass and delay lines.

This design has been tested and is working.
Parts:
- CN16: footprint Connector_PinHeader_2.00mm:PinHeader_2x22_P2.00mm_Vertical -> MyLibrary:IDE
- R721: footprint Resistor_SMD:R_1206_3216Metric_Pad1.42x1.75mm_HandSolder -> MyLibrary:SMD_1206
Connections:
- net labels added: +5V
- net labels removed: VCC
Other:
- note added: "Note: 14MHz or Vbb!"
- note added: "Warning:\nByte Swapped"
