File: Sheet12.sch (KiCad schematic (older format))
At the start: 35 parts, among them CN8 POWER

Commit message: Add files via upload
A slightly modified design, that removes the RF modulator and fits an S-Video connector in the space. It utilises the CXA2075 video encoder to create the S-video output and removes the need for the bandpass and delay lines.

This design has been tested and is working.
Parts:
- removed HL1, HL2, HL3: HOLE2, MyLibrary:Hole, symbol MyLibrary:HOLE2
- removed LFA1, LFB1, LFC1, LFD1: FB, MyLibrary:Filter, symbol Device:Ferrite_Bead_Small
- removed MT1, MT2, MT3, MT4: HOLE, MyLibrary:MT1-4, symbol MyLibrary:HOLE
- removed MT5: HOLE, MyLibrary:MT5, symbol MyLibrary:HOLE
- removed MT6: HOLE, MyLibrary:MT6, symbol MyLibrary:HOLE
- removed MT7: HOLE, MyLibrary:MT7, symbol MyLibrary:HOLE
- added H1, H2, H3: MountingHole, MyLibrary:Hole, symbol Mechanical:MountingHole
- added LF1: FERRITE, MyLibrary:Ferrite, symbol MyLibrary:FERRITE
- added MT1, MT2, MT3, MT4: MountingHole_Pad, MyLibrary:MT1-4, symbol Mechanical:MountingHole_Pad
- added MT5: MountingHole_Pad, MyLibrary:MT5, symbol Mechanical:MountingHole_Pad
- added MT6: MountingHole_Pad, MyLibrary:MT6, symbol Mechanical:MountingHole_Pad
- added MT7: MountingHole_Pad, MyLibrary:MT7, symbol Mechanical:MountingHole_Pad
- C800, C801, C802, C803: footprint Capacitor_SMD:C_1206_3216Metric_Pad1.42x1.75mm_HandSolder -> MyLibrary:SMD_1206
- C804: footprint Capacitor_SMD:C_1210_3225Metric_Pad1.42x2.65mm_HandSolder -> MyLibrary:SMD_1210
- C811: footprint Capacitor_THT:CP_Radial_D8.0mm_P5.00mm -> MyLibrary:C_RAD_P5
- C821, C822: footprint Capacitor_SMD:CP_Elec_6.3x5.9 -> MyLibrary:C_SMD_D6.3
- CN8: footprint MyLibrary:DS-215 -> MyLibrary:Power
- R952, RA951, RA953, RA954, RB951, RB953, RB954, RC951, RC953, RD951, RE951, RF951: footprint Resistor_SMD:R_1206_3216Metric_Pad1.42x1.75mm_HandSolder -> MyLibrary:SMD_1206
Connections:
- net labels added: +5V
- net labels removed: VCC
- wire segments 95 -> 90
Other:
- moved on the sheet: CN8, RA953, RA954, RB953, RB954, RC953
