File: Sheet2.sch (KiCad schematic (older format))
At the start: 39 parts, among them U16 256Kx16, U17 256Kx16, U25 74F258, U26 74F00, U27 74F139, X1 28.37516MHz

Commit message: Add files via upload
A slightly modified design, that removes the RF modulator and fits an S-Video connector in the space. It utilises the CXA2075 video encoder to create the S-video output and removes the need for the bandpass and delay lines.

This design has been tested and is working.
Parts:
- removed EC692, EC693: 47pF, Capacitor_SMD:C_1206_3216Metric_Pad1.42x1.75mm_HandSolder, symbol Device:C_Small
- removed ER131, ER692, ER693: 68, Resistor_SMD:R_1206_3216Metric_Pad1.42x1.75mm_HandSolder, symbol Device:R_Small
- removed U25: 74F258, Package_SO:SOIC-16_3.9x9.9mm_P1.27mm, symbol MyLibrary:74F258
- removed X1: 28.37516MHz, Oscillator:Oscillator_DIP-14, symbol MyLibrary:28.37516MHz
- added unit 2 of U16
- added unit 2 of U17
- added U25: 74F258, MyLibrary:SOIC-16-DUAL, symbol MyLibrary:74F258
- added unit 4 of U26
- added unit 3 of U26
- added unit 2 of U26
- added unit 2 of U27
- CA16, CA17, CB16, CB17: footprint Capacitor_SMD:C_1210_3225Metric_Pad1.42x2.65mm_HandSolder -> MyLibrary:SMD_1210
- E151: renamed from EC151; footprint Capacitor_SMD:C_1206_3216Metric_Pad1.42x1.75mm_HandSolder -> MyLibrary:SMD_1206
- E152: renamed from EC152; footprint Capacitor_SMD:C_1206_3216Metric_Pad1.42x1.75mm_HandSolder -> MyLibrary:SMD_1206
- E153: renamed from EC153; footprint Capacitor_SMD:C_1206_3216Metric_Pad1.42x1.75mm_HandSolder -> MyLibrary:SMD_1206
- E154: renamed from EC154; footprint Capacitor_SMD:C_1206_3216Metric_Pad1.42x1.75mm_HandSolder -> MyLibrary:SMD_1206
- EC150: footprint Capacitor_SMD:C_1206_3216Metric_Pad1.42x1.75mm_HandSolder -> MyLibrary:SMD_1206
- ER150, R161, RA151, RA152, RB151, RB152, RC151, RC152, RD151, RD152, RE151, RE152, RF151, RF152, RG151, RG152, RH151, RH152: footprint Resistor_SMD:R_1206_3216Metric_Pad1.42x1.75mm_HandSolder -> MyLibrary:SMD_1206
- R162: value * -> 470; footprint Resistor_SMD:R_1206_3216Metric_Pad1.42x1.75mm_HandSolder -> MyLibrary:SMD_1206
- U26: footprint Package_SO:SOIC-14_3.9x8.7mm_P1.27mm -> MyLibrary:SOIC-14
- U27: footprint Package_SO:SOIC-16_3.9x9.9mm_P1.27mm -> MyLibrary:SOIC-16-DUAL
Connections:
- net labels added: +5V
- net labels removed: CCK, U16_1, U16_20, U16_21, U16_35, U16_40, U16_6, U17_1, U17_20, U17_21, U17_35, U17_40, U17_6, U25_12, U25_16, U25_8, U26_14, U26_7, U27_16, U27_8, VCC, X1_1, X1_14, X1_7, XCLK, _CCK, _CCK_A
- wire segments 233 -> 198
- no-connect marks 0 -> 4
Other:
- note removed: "FUNNY INVERTERS"
- moved on the sheet: CA16, CA17, CB16, CB17, E151, E152, E153, E154, EC150, ER150, R161, R162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
