File: Sheet3.sch (KiCad schematic (older format))
At the start: 94 parts, among them CN10 RCA, Q211 2N3904, Q212 2N3904, Q213 2N3904, Q231 2N3904, Q232 2N3904, Q233 2N3904, Q461 2N3904, U12 CXA1145, U31 74HCT244, U32 74HCT244, U33 74LS74A, U4 DENISE, U50 CXA2075, X2 MODULATOR, Y451 4.433619MHz

Commit message: Add files via upload
A slightly modified design, that removes the RF modulator and fits an S-Video connector in the space. It utilises the CXA2075 video encoder to create the S-video output and removes the need for the bandpass and delay lines.

This design has been tested and is working.
Parts:
- removed C214: 10uF, Capacitor_SMD:CP_Elec_5x5.9, symbol Device:CP_Small
- removed C221, C222: 0.1uF, Capacitor_SMD:C_1206_3216Metric_Pad1.42x1.75mm_HandSolder, symbol Device:C_Small
- removed C235, C236, C239: 100uF, Capacitor_SMD:CP_Elec_6.3x5.9, symbol Device:CP_Small
- removed EC232: 0.01uF, Capacitor_SMD:C_1206_3216Metric_Pad1.42x1.75mm_HandSolder, symbol Device:C_Small
- removed ER232: 4.7, Resistor_SMD:R_2512_6332Metric_Pad1.52x3.35mm_HandSolder, symbol Device:R_Small
- removed Q211, Q212, Q213, Q231, Q232, Q233, Q461: 2N3904, Package_TO_SOT_SMD:SOT-23, symbol MyLibrary:TRANSISTOR
- removed R221: 1.2K/820, Resistor_SMD:R_1206_3216Metric_Pad1.42x1.75mm_HandSolder, symbol Device:R_Small
- removed R222: 1K, Resistor_SMD:R_1206_3216Metric_Pad1.42x1.75mm_HandSolder, symbol Device:R_Small
- removed R223: 1.2K/910, Resistor_SMD:R_1206_3216Metric_Pad1.42x1.75mm_HandSolder, symbol Device:R_Small
- removed R224: 820, Resistor_SMD:R_1206_3216Metric_Pad1.42x1.75mm_HandSolder, symbol Device:R_Small
- removed R225, R238: *, Resistor_SMD:R_1206_3216Metric_Pad1.42x1.75mm_HandSolder, symbol Device:R_Small
- removed R235: 360, Resistor_SMD:R_1206_3216Metric_Pad1.42x1.75mm_HandSolder, symbol Device:R_Small
- removed R236: 120/360, Resistor_SMD:R_1206_3216Metric_Pad1.42x1.75mm_HandSolder, symbol Device:R_Small
- removed R237: 100, Resistor_SMD:R_1206_3216Metric_Pad1.42x1.75mm_HandSolder, symbol Device:R_Small
- removed R975: 2.61K, Resistor_SMD:R_1206_3216Metric_Pad1.42x1.75mm_HandSolder, symbol Device:R_Small
- removed U50: CXA2075, MyLibrary:SOIC-24, symbol MyLibrary:CXA2075
- removed UJ50: Jumper, Jumper:SolderJumper-2_P1.3mm_Open_Pad1.0x1.5mm, symbol Device:Jumper_NO_Small
- removed X2: MODULATOR, MyLibrary:Modulator, symbol MyLibrary:MODULATOR
- removed Z221: BANDPASS, MyLibrary:Z221, symbol MyLibrary:BANDPASS
- removed Z222: DELAYLINE, MyLibrary:Z222, symbol MyLibrary:DELAYLINE
- added C281, C282: 220uF, MyLibrary:C_SMD_D6.3, symbol Device:CP_Small
- added Q211, Q212, Q213, Q231, Q232, Q233, Q461: 2N3904, MyLibrary:SOT-23, symbol MyLibrary:2N3904
- added R280: 2.61K, MyLibrary:SMD_1206, symbol Device:R_Small
- added R281, R282: 75, MyLibrary:SMD_1206, symbol Device:R_Small
- added RE234: 240, MyLibrary:SMD_1206, symbol Device:R_Small
- added unit 2 of U33
- added X2: MINI-DIN, MyLibrary:S-Video, symbol MyLibrary:MINI-DIN
- C201: footprint MyLibrary:TZ03 -> MyLibrary:Trimmer; symbol Device:C_Variable -> Device:CTRIM_Small
- C211, C212, C213: footprint Capacitor_SMD:C_1210_3225Metric_Pad1.42x2.65mm_HandSolder -> MyLibrary:SMD_1210
- C237: value 470uF -> 220uF; footprint Capacitor_THT:CP_Radial_D8.0mm_P5.00mm -> MyLibrary:C_SMD_D6.3
- C241, C242, C243, C244, C245, C246, EC231: footprint Capacitor_SMD:C_1206_3216Metric_Pad1.42x1.75mm_HandSolder -> MyLibrary:SMD_1206
- ER231: value 100 -> FB100; footprint Resistor_SMD:R_1206_3216Metric_Pad1.42x1.75mm_HandSolder -> MyLibrary:SMD_1206
- L241: footprint Inductor_SMD:L_1206_3216Metric_Pad1.42x1.75mm_HandSolder -> MyLibrary:SMD_1210
- R202, R203, R211, R212, R213, R241, R242, R243, R244, R245, R246, RA214, RA215, RA216, RA231, RA232, RA233, RA234, RB214, RB215, RB216, RB231, RB232, RB233, RB234, RC214, RC215, RC216, RC231, RC232, RC233, RC234, RD214, RD215, RD216, RE214, RE215, RE216, RE232, RF214, RF215, RF216: footprint Resistor_SMD:R_1206_3216Metric_Pad1.42x1.75mm_HandSolder -> MyLibrary:SMD_1206
- RD234: value 75 -> 43; footprint Resistor_SMD:R_1206_3216Metric_Pad1.42x1.75mm_HandSolder -> MyLibrary:SMD_1206
- U12: value CXA1145 -> CXA2075M; footprint MyLibrary:SOIC-24 -> MyLibrary:SOP-24; symbol MyLibrary:CXA1145 -> MyLibrary:CXA2075M
- U31, U32: footprint Package_SO:SOIC-20W_7.5x12.8mm_P1.27mm -> MyLibrary:SOIC-20W
- U33: footprint Package_SO:SOIC-14_3.9x8.7mm_P1.27mm -> MyLibrary:SOIC-14
- U4: footprint Package_LCC:PLCC-52 -> MyLibrary:PLCC-52
- Y451: symbol Amiga600-rescue:Crystal_GND3_Small-Device -> Device:Crystal_GND3_Small
Connections:
- net labels added: +5V
- net labels removed: MONO, U12_1, U12_12, U12_13, U12_14, U12_19, U12_24, U31_10, U31_20, U32_10, U32_20, U33_14, U33_7, U4_21, U4_40, U50_1, U50_12, U50_19, U50_24, VCC, VVref
- wire segments 394 -> 276
- no-connect marks 7 -> 1
Other:
- note added: "1% tolerance"
- note added: "CC@4"
- note added: "Note: NTSC\nuses 3.32K\n\n1% tolerance"
- note added: "R202 = NTSC\nR203 = PAL"
- note added: "S-VIDEO"
- note removed: "MODULATOR"
- moved on the sheet: C211, C212, C213, C237, C241, C242, C243, C244, C245, C246, CN10, EC231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
