File: Sheet4.sch (KiCad schematic (older format))
At the start: 97 parts, among them CN1 DB9P, CN2 DB9P, CN3 RCA, CN4 RCA, Q321 MPF102, Q331 MPF102, Q341 2N3906, U15 TL084, U3 PAULA, U34 74LS157

Commit message: Add files via upload
A slightly modified design, that removes the RF modulator and fits an S-Video connector in the space. It utilises the CXA2075 video encoder to create the S-video output and removes the need for the bandpass and delay lines.

This design has been tested and is working.
Parts:
- removed Q321, Q331: MPF102, Package_TO_SOT_SMD:SOT-23, symbol MyLibrary:TRANSISTOR
- removed Q341: 2N3906, Package_TO_SOT_SMD:SOT-23, symbol MyLibrary:TRANSISTOR
- added Q321, Q331: MPF102, MyLibrary:SOT-23, symbol MyLibrary:MPF102
- added Q341: 2N3906, MyLibrary:SOT-23, symbol MyLibrary:2N3906
- added unit 2 of U15
- added unit 4 of U15
- added unit 3 of U15
- added U28: 1488, MyLibrary:SOIC-14, symbol MyLibrary:1488
- C311, C312, C313, C314: value 0.047pF -> 0.047uF; footprint Capacitor_SMD:C_1206_3216Metric_Pad1.42x1.75mm_HandSolder -> MyLibrary:SMD_1206
- C321, C322, C323, C331, C332, C333, C349, C352, C362, EC351, EC353, EC354, EC355, EC356, EC357, EC358, EC361, EC363, EC364, EC365, EC366, EC367, EC368, EC371, EC372, EC373, EC374: footprint Capacitor_SMD:C_1206_3216Metric_Pad1.42x1.75mm_HandSolder -> MyLibrary:SMD_1206
- C324, C334: footprint Capacitor_SMD:CP_Elec_6.3x5.9 -> MyLibrary:C_SMD_D6.3
- EC321, EC331: value 6800 -> 6800pF; footprint Capacitor_SMD:C_1206_3216Metric_Pad1.42x1.75mm_HandSolder -> MyLibrary:SMD_1206
- ER321, ER331, ER351, ER353, ER354, ER355, ER356, ER357, ER358, ER361, ER363, ER364, ER365, ER366, ER367, ER368, ER371, ER372, ER373, ER374, R319, R322, R323, R324, R325, R326, R327, R329, R332, R333, R334, R335, R336, R337, R339, R345, R346, R347, R348, R349, RA370, RB370, RC370, RD370, RE370, RF370, RG370, RH370: footprint Resistor_SMD:R_1206_3216Metric_Pad1.42x1.75mm_HandSolder -> MyLibrary:SMD_1206
- R321, R331: value 1.5K -> 680; footprint Resistor_SMD:R_1206_3216Metric_Pad1.42x1.75mm_HandSolder -> MyLibrary:SMD_1206
- R352, R362: footprint Resistor_SMD:R_2512_6332Metric_Pad1.52x3.35mm_HandSolder -> MyLibrary:SMD_2512
- U15: footprint Package_SO:SOIC-14_3.9x8.7mm_P1.27mm -> MyLibrary:SOIC-14
- U3: footprint Package_LCC:PLCC-52 -> MyLibrary:PLCC-52
- U34: footprint Package_SO:SOIC-16_3.9x9.9mm_P1.27mm -> MyLibrary:SOIC-16
Connections:
- net labels added: +5V, AUDIO, AVREF, _LED, _RXD, _TXD
- net labels removed: AVref, GNDA, U15_11, U15_4, U28_3, U34_16, U34_8, U3_30, U3_37, U3_8, VCC, _RxD, _TxD
- wire segments 380 -> 362
Other:
- note added: "Note: LED off, Filters bypassed"
- moved on the sheet: C321, C331, C333, C352, C362, EC321, EC331, EC355, EC356, EC357, EC358, EC365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
