File: Sheet5.sch (KiCad schematic (older format))
At the start: 83 parts, among them CN9 DB23P

Commit message: Add files via upload
A slightly modified design, that removes the RF modulator and fits an S-Video connector in the space. It utilises the CXA2075 video encoder to create the S-video output and removes the need for the bandpass and delay lines.

This design has been tested and is working.
Parts:
- removed C458, C461: 0.01uF, Capacitor_SMD:C_1206_3216Metric_Pad1.42x1.75mm_HandSolder, symbol Device:C_Small
- removed C459: 22uF, Capacitor_SMD:CP_Elec_5x5.9, symbol Device:CP_Small
- removed C460: 10uF, Capacitor_SMD:CP_Elec_5x5.9, symbol Device:CP_Small
- removed R459: 27K, Resistor_SMD:R_1206_3216Metric_Pad1.42x1.75mm_HandSolder, symbol Device:R_Small
- added U1: MC68000, MyLibrary:PLCC-68, symbol MyLibrary:MC68000
- added U12: CXA2075M, MyLibrary:SOP-24, symbol MyLibrary:CXA2075M
- added U15: TL084, MyLibrary:SOIC-14, symbol MyLibrary:TL084
- added U2: AGNUS, MyLibrary:PLCC-84, symbol MyLibrary:AGNUS
- added U21, U22: 74LS245, MyLibrary:SOIC-20W, symbol MyLibrary:74LS245
- added U25: 74F258, MyLibrary:SOIC-16-DUAL, symbol MyLibrary:74F258
- added U26: 74F00, MyLibrary:SOIC-14, symbol MyLibrary:74F00
- added U27: 74F139, MyLibrary:SOIC-16-DUAL, symbol MyLibrary:74F139
- added U3: PAULA, MyLibrary:PLCC-52, symbol MyLibrary:PAULA
- added U31, U32: 74HCT244, MyLibrary:SOIC-20W, symbol MyLibrary:74HCT244
- added U33: 74LS74A, MyLibrary:SOIC-14, symbol MyLibrary:74LS74A
- added U34: 74LS157, MyLibrary:SOIC-16, symbol MyLibrary:74LS157
- added U4: DENISE, MyLibrary:PLCC-52, symbol MyLibrary:DENISE
- added U5: GAYLE, MyLibrary:PLCC-84, symbol MyLibrary:GAYLE
- added X1: 28.37516MHz, MyLibrary:Oscillator, symbol MyLibrary:28.37516MHz
- C199, C2, C21, C22, C25, C3, C301, C302, C305, C31, C32, C4, CA1, CA12, CA5, CB1, CB12, CB5: footprint Capacitor_SMD:C_1210_3225Metric_Pad1.42x2.65mm_HandSolder -> MyLibrary:SMD_1210
- C26, C27, C33, C34: value 0.047uF -> 0.01uF; footprint Capacitor_SMD:C_1206_3216Metric_Pad1.42x1.75mm_HandSolder -> MyLibrary:SMD_1206
- C303, C304, C409: footprint Capacitor_SMD:CP_Elec_6.3x5.9 -> MyLibrary:C_SMD_D6.3
- C306: footprint Capacitor_SMD:CP_Elec_5x5.9 -> MyLibrary:C_SMD_D5
- C307, C408: footprint Capacitor_THT:CP_Radial_D8.0mm_P5.00mm -> MyLibrary:C_RAD_P5
- E301, FB991, FB992: footprint Resistor_SMD:R_1812_4532Metric_Pad1.30x3.40mm_HandSolder -> MyLibrary:SMD_1812
- EC251, EC252, EC253, EC254, EC255, EC256, EC257, EC258, EC259, EC260, EC261, EC262, EC263, EC264, EC265, EC266, EC267: footprint Capacitor_SMD:C_1206_3216Metric_Pad1.42x1.75mm_HandSolder -> MyLibrary:SMD_1206
- ER251, ER252, ER253, ER254, ER255, ER256, ER257, ER261, ER262, ER266, ER267, R251, R252, R253, R301, R302, R303, R304: footprint Resistor_SMD:R_1206_3216Metric_Pad1.42x1.75mm_HandSolder -> MyLibrary:SMD_1206
- ER258, ER259, ER260, ER263, ER264, ER265: value 200 -> FB200; footprint Resistor_SMD:R_1206_3216Metric_Pad1.42x1.75mm_HandSolder -> MyLibrary:SMD_1206
- FB993: footprint Resistor_SMD:R_1812_4532Metric_Pad1.30x3.40mm_HandSolder -> MyLibrary:SMD_1206
- R309, R406, RA405, RB405: footprint Resistor_SMD:R_2512_6332Metric_Pad1.52x3.35mm_HandSolder -> MyLibrary:SMD_2512
Connections:
- net labels added: +5V, AUDIO, AVREF
- net labels removed: AVref, GNDA, U12_1, U12_12, U12_13, U12_14, U12_19, U12_24, U15_11, U15_4, U1_14, U1_16, U1_17, U1_18, U1_31, U1_52, U1_56, U1_57, U21_10, U21_20, U22_10, U22_20, U25_16, U25_8, U26_14, U26_7, U27_16, U27_8, U2_15, U2_41, U2_58, U2_82, U31_10, U31_20, U32_10, U32_20, U33_14, U33_7, U34_16, U34_8, U3_30, U3_37, U3_8, U4_21, U4_40, U50_1, U50_12, U50_19, U50_24, U5_20, U5_24, U5_3, U5_45, U5_62, U5_66, VCC, VVref, X1_1, X1_14, X1_7
- wire segments 383 -> 304
Other:
- note added: "AUDIO DECOUPLING"
- note added: "Note: Ground interconnection near audio jacks."
- note removed: "DECOUPLING"
- moved on the sheet: C199, C2, C21, C22, C25, C26, C27, C3, C301, C302, C303, C304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
