File: Sheet6.sch (KiCad schematic (older format))
At the start: 71 parts, among them CN6 DB25P, CN7 DB25S, Q571 2N3904, U28 1488, U29 1489, U7 8520, U8 8520

Commit message: Add files via upload
A slightly modified design, that removes the RF modulator and fits an S-Video connector in the space. It utilises the CXA2075 video encoder to create the S-video output and removes the need for the bandpass and delay lines.

This design has been tested and is working.
Parts:
- removed D571: 1N914, Package_TO_SOT_SMD:SOT-23, symbol MyLibrary:TRANSISTOR
- removed Q571: 2N3904, Package_TO_SOT_SMD:SOT-23, symbol MyLibrary:TRANSISTOR
- added D571: 1N914, MyLibrary:SOT-23_Diode, symbol Device:D_Small
- added Q571: 2N3904, MyLibrary:SOT-23, symbol MyLibrary:2N3904
- added unit 3 of U28
- added unit 2 of U28
- added unit 4 of U29
- added unit 2 of U29
- added unit 3 of U29
- C551, C552: footprint Capacitor_SMD:C_1210_3225Metric_Pad1.42x2.65mm_HandSolder -> MyLibrary:SMD_1210
- D572, D573, D574: footprint Diode_SMD:D_MELF -> MyLibrary:SMD_MELF
- EC511, EC512, EC513, EC514, EC515, EC516, EC517, EC518, EC519, EC520, EC521, EC522, EC523, EC524, EC525, EC551, EC552, EC553, EC554, EC555, EC556, EC557, EC558, EC561, EC562: footprint Capacitor_SMD:C_1206_3216Metric_Pad1.42x1.75mm_HandSolder -> MyLibrary:SMD_1206
- ER511, ER512, ER517, ER518, ER519, ER520, ER521, ER522, ER523, ER525, ER551, ER552, ER553, ER554, ER555, ER556, ER557, ER558, ER561, ER562, R512, R571, R572, RA511, RB511, RC511, RF511, RI511: footprint Resistor_SMD:R_1206_3216Metric_Pad1.42x1.75mm_HandSolder -> MyLibrary:SMD_1206
- ER513, ER514, ER515, ER516: value 47 -> 68; footprint Resistor_SMD:R_1206_3216Metric_Pad1.42x1.75mm_HandSolder -> MyLibrary:SMD_1206
- ER524: footprint Resistor_SMD:R_2512_6332Metric_Pad1.52x3.35mm_HandSolder -> MyLibrary:SMD_2512
- U28, U29: footprint Package_SO:SOIC-14_3.9x8.7mm_P1.27mm -> MyLibrary:SOIC-14
- U7, U8: footprint Package_LCC:PLCC-44 -> MyLibrary:PLCC-44
Connections:
- net labels added: +5V, _RXD, _TXD
- net labels removed: U28_1, U28_14, U28_3, U28_7, U29_14, U29_7, U7_1, U7_22, U8_1, U8_22, VCC, _RxD, _TxD
- wire segments 319 -> 307
- no-connect marks 16 -> 15
Other:
- note added: "OPTIONAL"
- moved on the sheet: D572, D573, D574, R512, R571, R572, RA511, RB511, RC511, RF511, RI511, U29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
