File: Sheet7.sch (KiCad schematic (older format))
At the start: 52 parts, among them CN11 FLOPPY, CN12 4PIN, CN5 DB23S

Commit message: Add files via upload
A slightly modified design, that removes the RF modulator and fits an S-Video connector in the space. It utilises the CXA2075 video encoder to create the S-video output and removes the need for the bandpass and delay lines.

This design has been tested and is working.
Parts:
- added U28: 1488, MyLibrary:SOIC-14, symbol MyLibrary:1488
- added U29: 1489, MyLibrary:SOIC-14, symbol MyLibrary:1489
- added U5: GAYLE, MyLibrary:PLCC-84, symbol MyLibrary:GAYLE
- added U7, U8: 8520, MyLibrary:PLCC-44, symbol MyLibrary:8520
- C29, C7, C8, CA28, CB28: value 0.047uF -> 0.01uF; footprint Capacitor_SMD:C_1206_3216Metric_Pad1.42x1.75mm_HandSolder -> MyLibrary:SMD_1206
- C591, C592, EC580, EC581, EC582, EC583, EC584, EC585, EC586, EC587, EC588, EC589, EC590, EC591, EC592, EC593, EC594, EC595, EC596, EC597, EC598, EC599: footprint Capacitor_SMD:C_1206_3216Metric_Pad1.42x1.75mm_HandSolder -> MyLibrary:SMD_1206
- CN11: footprint Connector_PinHeader_2.54mm:PinHeader_2x17_P2.54mm_Vertical -> MyLibrary:Floppy
- CN12: footprint Connector_PinHeader_2.54mm:PinHeader_1x04_P2.54mm_Vertical -> MyLibrary:1x04_P2.54
- D575, D576: footprint Diode_SMD:D_MELF -> MyLibrary:SMD_MELF
- ER580, ER581, ER582, ER583, ER584, ER585, ER586, ER587, ER588, ER589, ER590, ER591, ER592, ER593, ER594, ER595, ER596, ER599: footprint Resistor_SMD:R_1206_3216Metric_Pad1.42x1.75mm_HandSolder -> MyLibrary:SMD_1206
- ER597, ER598: value 200 -> FB200; footprint Resistor_SMD:R_1206_3216Metric_Pad1.42x1.75mm_HandSolder -> MyLibrary:SMD_1206
Connections:
- net labels added: +5V
- net labels removed: U28_1, U28_14, U28_7, U29_14, U29_7, U5_63, U5_64, U5_65, U5_67, U5_68, U5_69, U5_70, U5_71, U5_72, U7_1, U7_22, U8_1, U8_22, VCC
- wire segments 247 -> 246
Other:
- note added: "EXTERNAL FLOPPY"
- note added: "Note: Some drives are +5 only..."
- moved on the sheet: C29, C591, C592, C7, C8, CA28, CB28, CN11, CN12, CN5, D575, D576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
