File: Sheet8.sch (KiCad schematic (older format))
At the start: 42 parts, among them CN13 KEYBOARD, CN14 4PIN, Q511 2N3904, Q621 2N3904, Q622 2N3904, Q631 2N3906, Q632 2N3906, Q633 2N3906, Q634 *, U13 6570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

Commit message: Add files via upload
A slightly modified design, that removes the RF modulator and fits an S-Video connector in the space. It utilises the CXA2075 video encoder to create the S-video output and removes the need for the bandpass and delay lines.

This design has been tested and is working.
Parts:
- removed Q511, Q621, Q622: 2N3904, Package_TO_SOT_SMD:SOT-23, symbol MyLibrary:TRANSISTOR
- removed Q631, Q632, Q633: 2N3906, Package_TO_SOT_SMD:SOT-23, symbol MyLibrary:TRANSISTOR
- removed Q634: *, Package_TO_SOT_SMD:SOT-23, symbol MyLibrary:TRANSISTOR
- removed U49: TC54VN43, Package_TO_SOT_SMD:SOT-23, symbol MyLibrary:TRANSISTOR
- added Q511, Q621, Q622: 2N3904, MyLibrary:SOT-23, symbol MyLibrary:2N3904
- added Q631, Q632, Q633, Q634: 2N3906, MyLibrary:SOT-23, symbol MyLibrary:2N3906
- added unit 2 of U13
- added unit 2 of U14
- added unit 2 of U36
- added U49: RH5VA43A, MyLibrary:SOT-89, symbol MyLibrary:RH5VA43A
- C13, C14: footprint Capacitor_SMD:C_1210_3225Metric_Pad1.42x2.65mm_HandSolder -> MyLibrary:SMD_1210
- C36: value 0.047uF -> 0.01uF; footprint Capacitor_SMD:C_1206_3216Metric_Pad1.42x1.75mm_HandSolder -> MyLibrary:SMD_1206
- C611, C613: footprint Capacitor_SMD:C_1206_3216Metric_Pad1.42x1.75mm_HandSolder -> MyLibrary:SMD_1206
- C612: footprint Capacitor_SMD:CP_Elec_5x5.9 -> MyLibrary:C_SMD_D5
- C621, C622: value 22pF* -> 22pF; footprint Capacitor_SMD:C_1206_3216Metric_Pad1.42x1.75mm_HandSolder -> MyLibrary:SMD_1206
- CN14: footprint Connector_PinHeader_2.54mm:PinHeader_1x04_P2.54mm_Vertical -> MyLibrary:1x04_P2.54
- R514, R515, R611, R612, R621, R622, R623, R624, R625, R626, R631, R632, R633, R634, R635, R636, R639, RD511: footprint Resistor_SMD:R_1206_3216Metric_Pad1.42x1.75mm_HandSolder -> MyLibrary:SMD_1206
- R637: value * -> 10K; footprint Resistor_SMD:R_1206_3216Metric_Pad1.42x1.75mm_HandSolder -> MyLibrary:SMD_1206
- R638: value * -> 4.7K; footprint Resistor_SMD:R_1206_3216Metric_Pad1.42x1.75mm_HandSolder -> MyLibrary:SMD_1206
- U13: footprint Package_LCC:PLCC-44 -> MyLibrary:PLCC-44
- U14: footprint Package_SO:SOIC-8_3.9x4.9mm_P1.27mm -> MyLibrary:SOIC-8
- U36: footprint Package_SO:SOIC-14_3.9x8.7mm_P1.27mm -> MyLibrary:SOIC-14
Connections:
- net labels added: +5V
- net labels removed: U13_1, U13_13, U13_33, U14_1, U14_8, U36_14, U36_7, VCC
- wire segments 210 -> 196
Other:
- note added: "OPTIONAL"
- note added: "U49 added Rev 2C"
- moved on the sheet: C13, C14, C36, C611, C612, C613, C621, C622, CN14, R514, R515, R611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
