File: Sheet9.sch (KiCad schematic (older format))
At the start: 24 parts, among them CN17 7PIN, Q502 2N3906, Q503 2N3906, Q651 2N3904, Q652 2N3906, Q653 2N3904, Q654 2N3906, U6 ROM

Commit message: Add files via upload
A slightly modified design, that removes the RF modulator and fits an S-Video connector in the space. It utilises the CXA2075 video encoder to create the S-video output and removes the need for the bandpass and delay lines.

This design has been tested and is working.
Parts:
- removed CN17: 7PIN, MyLibrary:Keyboard, symbol MyLibrary:7PIN
- removed Q502, Q503, Q652, Q654: 2N3906, Package_TO_SOT_SMD:SOT-23, symbol MyLibrary:TRANSISTOR
- removed Q651, Q653: 2N3904, Package_TO_SOT_SMD:SOT-23, symbol MyLibrary:TRANSISTOR
- removed R503, R504: 4.7K, Resistor_SMD:R_1206_3216Metric_Pad1.42x1.75mm_HandSolder, symbol Device:R_Small
- removed R505, R506: 10K, Resistor_SMD:R_1206_3216Metric_Pad1.42x1.75mm_HandSolder, symbol Device:R_Small
- removed R507: 100, Resistor_SMD:R_1206_3216Metric_Pad1.42x1.75mm_HandSolder, symbol Device:R_Small
- added EC692, EC693: 47pF, MyLibrary:SMD_1206, symbol Device:C_Small
- added ER692, ER693: 68, MyLibrary:SMD_1206, symbol Device:R_Small
- added Q651, Q653: 2N3904, MyLibrary:SOT-23, symbol MyLibrary:2N3904
- added Q652, Q654: 2N3906, MyLibrary:SOT-23, symbol MyLibrary:2N3906
- added U25: 74F258, MyLibrary:SOIC-16-DUAL, symbol MyLibrary:74F258
- added unit 2 of U6
- C6: footprint Capacitor_SMD:C_1210_3225Metric_Pad1.42x2.65mm_HandSolder -> MyLibrary:SMD_1210
- R651, R652, R653, R654, R655, R656, R657, R658, R659, R660: footprint Resistor_SMD:R_1206_3216Metric_Pad1.42x1.75mm_HandSolder -> MyLibrary:SMD_1206
- U6: footprint Package_DIP:DIP-42_W15.24mm -> MyLibrary:DIP-42
Connections:
- net labels added: +5V, CCK, VPP, _CCK, _CCK_A, _XCLKEN
- net labels removed: U6_12, U6_22, U6_31, VCC, Vpp, _KB_CLOCK, _KB_DATA, _KB_RESET, _LED, _MTR0
- wire segments 117 -> 100
- no-connect marks 0 -> 1
Other:
- note added: "FUNNY INVERTERS"
- note removed: "A500 KEYBOARD CONNECTOR"
- moved on the sheet: C6, R651, R652, R653, R654, R655, R656, R657, R658, R659, R660
